File: PneuDis_HuskReel_SCH.sch (KiCad schematic (older format))
At the start: 7 parts

Commit message: Update
Parts:
- removed CB?: CircuitBreaker_1P_US, symbol Build_002K-rescue:CircuitBreaker_1P_US
- removed K?: AUTOMOTIVE_STD_RELAY_SPST, symbol Build_002K-rescue:AUTOMOTIVE_STD_RELAY_SPST
- removed SW? (x2): SW_PUSHBUTTON-freetronics_schematic-Draft_001-res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, symbol Build_002K-rescue:SW_PUSHBUTTON-freetronics_schematic-Draft_001-rescue-Draft-re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
- removed U?: WAYTEK75610, symbol Build_002K-rescue:WAYTEK75610
- added CB?: EATON 122A30-00M-KA, symbol Build_002K-rescue:CircuitBreaker_1P_US
- added J? (x3): Conn_01x02_Female, symbol Connector:Conn_01x02_Female
- added J? (x3): Conn_01x02_Male, symbol Connector:Conn_01x02_Male
- added J?: F CONN 19436-0213, symbol Connector:Conn_01x02_Female
- added J?: M CONN 19432-0013, symbol Connector:Conn_01x02_Male
- added K?: AUTOMOTIVE_STD_RELAY_SPST, symbol Build_002K-rescue:AUTOMOTIVE_STD_RELAY_SPST
- added SW? (x2): SW_PUSHBUTTON, symbol Build_002K-rescue:SW_PUSHBUTTON
- added U? (x2): WAYTEK75610, symbol Build_002K-rescue:WAYTEK75610
Connections:
- net at BT?.1 (+): now also CB?.2
- net at BT?.2 (-): now also J?.1 (Pin_1)
- net at M?.1 (+): now also J?.2 (Pin_2)
- net at M?.2 (-): now also J?.1 (Pin_1)
- new net: J?.1 (Pin_1), SW?.2 (x2)
- new net: J?.2 (Pin_2), SW?.1 (x2)
- new net: CB?.1, J?.2 (Pin_2)
- new net: J?.1 (Pin_1), J?.1 (Pin_1), J?.2 (Pin_2), U?.30
- new net: J?.2 (Pin_2), J?.2 (Pin_2), U?.85
- new net: J?.1 (Pin_1), J?.1 (Pin_1), U?.86
- new net: J?.2 (Pin_2), U?.87
- no-connect marks 0 -> 7
Other:
- note added: "20" 10G RED"
- note added: "20" 20G BLACK"
- note added: "20" 20G RED"
- note added: "27" 10G BLACK"
- note added: "3" 12G RED"
- note added: "3" 18G BLACK"
- note added: "3" 20G BLACK"
- note added: "3" 20G RED"
- note added: "3.5" 18G BLUE"
- note added: "30564 Vinyl Male Bullet Connector\n\n"
- note added: "30565 Vinyl Female Bullet Connector\n\n"
- note added: "5" 10G RED"
- note added: "5/16 RING TERMINAL"
- note added: "6" 10G BLACK"
- note added: "6" 10G RED"
- note added: "6" 20G BLACK"
- note added: "81" 10G BLACK"
- note added: "81" 10G RED"
- note added: "821240\nSplice"
- note added: "Aptvi 5-PIN Connector 75612\n12066614 F TERM 16G\n12033997 F TERM 10G"
- note added: "MIZU-P25\n52213-0211 - RECEPT\n50148-8000 - F TERMINAL"
- note added: "MIZU-P25\n52266-0211 - PLUG\n50147-8000 - M TERMINAL"
- note added: "Molex 19432-0013\n194310016 - M TERM"
- note added: "Molex 19436-0213\n194340003 - F TERM"
- moved on the sheet: M?

Commit message: Update
Parts:
- removed J?: Conn_01x02_Female, symbol Connector:Conn_01x02_Female
- removed J?: Conn_01x02_Male, symbol Connector:Conn_01x02_Male
- added CB?: EATON 122A30-00M-KA, symbol Build_002K-rescue:CircuitBreaker_1P_US
- added J? (x2): Conn_01x01_Female, symbol Connector:Conn_01x01_Female
- added J? (x2): Conn_01x01_Male, symbol Connector:Conn_01x01_Male
- added J?: M CONN 19432-0013, symbol Connector:Conn_01x02_Male
- added J?: F CONN 19436-0213, symbol Connector:Conn_01x02_Female
Connections:
- net at M?.1 (+): now also J?.2 (Pin_2)
- net at M?.2 (-): now also J?.1 (Pin_1)
- net at SW?.1: now also J?.1 (Pin_1); no longer J?.2 (Pin_2)
- net at SW?.2: now also J?.2 (Pin_2); no longer J?.1 (Pin_1)
- net at J?.2 (Pin_2), U?.85: now also J?.2 (Pin_2); no longer J?.2 (Pin_2)
- net at U?.86: now also J?.1 (Pin_1), J?.1 (Pin_1); no longer J?.1 (Pin_1)
- net at U?.87: now also J?.1 (Pin_1), J?.1 (Pin_1), J?.2 (Pin_2)
- new net: J?.1 (Pin_1), U?.30
- new net: J?.1 (Pin_1), J?.1 (Pin_1)
- new net: J?.1 (Pin_1), J?.2 (Pin_2)
- no-connect marks 7 -> 4
Other:
- note added: "3/4 Conduit"
- note added: "3/4 Plastic Conduit"
- note added: "Female Spade Connector\n\n"
- note added: "Male Spade Connector\n\n"
- note removed: "20" 20G BLACK"
- note removed: "20" 20G RED"
- note removed: "3" 12G RED"
- note removed: "3" 18G BLACK"
- note removed: "3" 20G BLACK"
- note removed: "3" 20G RED"
- note removed: "3.5" 18G BLUE"
- note removed: "30564 Vinyl Male Bullet Connector\n\n"
- note removed: "30565 Vinyl Female Bullet Connector\n\n"
- note removed: "5" 10G RED"
- note removed: "821240\nSplice"
- moved on the sheet: BT?, J?, K?
